File: kicad/MP1.kicad_pcb (KiCad board)
At the start: 2 copper layers, 16.1 x 14 mm, 14 parts, among them J1 48037-0001, U1 MCP1702T-3302E_CB, U2 MCP6021T-E_OT

Commit message: Tidy silkscreen and fab layers; full design-choice report; drop unused LTspice draft
- F.SilkS: labels off pads, plug's off-board body outline removed
- F.Fab: 0.5 mm values beside parts, reference text in IC/connector bodies
- B.SilkS: title / author / revision block
- Library footprints for J1, U1, U2 updated to match the board
- Report: every circuit and PCB design choice explained, BOM table added
Other:
- board text added: "D. SHAH ENGR 3430"
- board text added: "MP1 LED FLASHER"
- board text added: "REV A 2026-09"
Changed lines of the file:
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@@
 		(tags "capacitor")
 		(property "Reference" "C4"
-			(at -0.6 1.405 0)
+			(at -1.75 1.355 90)
 			(unlocked yes)
 			(layer "F.SilkS")
@@
 		)
 		(property "Value" "0.1u"
-			(at 0 1.43 0)
-			(layer "F.Fab")
-			(effects
-				(font
-					(size 1 1)
-					(thickness 0.15)
+			(at -2.05 0.505 90)
+			(unlocked yes)
+			(layer "F.Fab")
+			(effects
+				(font
+					(size 0.5 0.5)
+					(thickness 0.08)
 				)
 			)
@@
 		(tags "resistor")
 		(property "Reference" "R3"
-			(at -2 0 0)
+			(at -1.75 0 90)
 			(unlocked yes)
 			(layer "F.SilkS")
@@
 		)
 		(property "Value" "40.2k"
-			(at 0 1.43 0)
-			(layer "F.Fab")
-			(effects
-				(font
-					(size 1 1)
-					(thickness 0.15)
+			(at -2.05 -0.2 90)
+			(unlocked yes)
+			(layer "F.Fab")
+			(effects
+				(font
+					(size 0.5 0.5)
+					(thickness 0.08)
 				)
 			)
@@
 		(at 123 106.4 -90)
 		(property "Reference" "U2"
-			(at 0 1.8 90)
+			(at 0.25 1.7 90)
 			(unlocked yes)
 			(layer "F.SilkS")
@@
 		)
 		(property "Value" "MCP6021T-E_OT"
-			(at 8.105 3.335 90)
-			(layer "F.Fab")
-			(effects
-				(font
-					(size 1 1)
-					(thickness 0.15)
+			(at -0.5 -2.45 90)
+			(unlocked yes)
+			(layer "F.Fab")
+			(effects
+				(font
+					(size 0.4 0.4)
+					(thickness 0.08)
 				)
 			)
@@
 			(fill no)
 			(layer "F.Fab")
+		)
+		(fp_text user "${REFERENCE}"
+			(at 0 0 90)
+			(unlocked yes)
+			(layer "F.Fab")
+			(effects
+				(font
+					(size 0.5 0.5)
+					(thickness 0.08)
+				)
+			)
 		)
 		(pad "1" smd roundrect
@@
 		)
 		(property "Value" "3.01M"
-			(at 0 1.43 0)
-			(layer "F.Fab")
-			(effects
-				(font
-					(size 1 1)
-					(thickness 0.15)
+			(at 1.95 0.15 90)
+			(unlocked yes)
+			(layer "F.Fab")
+			(effects
+				(font
+					(size 0.5 0.5)
+					(thickness 0.08)
 				)
 			)
@@
 		(tags "LED")
 		(property "Reference" "D1"
-			(at -2.25 0.25 90)
+			(at -2.2 0.4 90)
 			(unlocked yes)
 			(layer "F.SilkS")
@@
 		)
 		(property "Value" "LED"
-			(at 0 1.65 0)
-			(layer "F.Fab")
-			(effects
-				(font
-					(size 1 1)
-					(thickness 0.15)
+			(at -1.4 0 90)
+			(unlocked yes)
+			(layer "F.Fab")
+			(effects
+				(font
+					(size 0.5 0.5)
+					(thickness 0.08)
 				)
 			)
@@
 		(at 118.7 112.1 90)
 		(property "Reference" "U1"
-			(at 2.5 -1.2 0)
+			(at -1.1 -2 90)
 			(unlocked yes)
 			(layer "F.SilkS")
@@
 		)
 		(property "Value" "MCP1702T-3302E_CB"
-			(at 10.93553 3.25523 90)
-			(layer "F.Fab")
-			(effects
-				(font
-					(size 1.642031 1.642031)
-					(thickness 0.15)
+			(at 0 -2 90)
+			(unlocked yes)
+			(layer "F.Fab")
+			(effects
+				(font
+					(size 0.4 0.4)
+					(thickness 0.08)
 				)
 			)
@@
 			)
 			(layer "F.Fab")
+		)
+		(fp_text user "${REFERENCE}"
+			(at 0 0 90)
+			(unlocked yes)
+			(layer "F.Fab")
+			(effects
+				(font
+					(size 0.5 0.5)
+					(thickness 0.08)
+				)
+			)
 		)
 		(pad "1" smd rect
@@
 		(tags "resistor")
 		(property "Reference" "R2"
-			(at 0 -1.275 90)
+			(at 0 -1.195 90)
 			(unlocked yes)
 			(layer "F.SilkS")
@@
 		)
 		(property "Value" "4.99k"
-			(at 0 1.43 270)
-			(layer "F.Fab")
-			(effects
-				(font
-					(size 1 1)
-					(thickness 0.15)
+			(at 0 -1.225 90)
+			(unlocked yes)
+			(layer "F.Fab")
+			(effects
+				(font
+					(size 0.5 0.5)
+					(thickness 0.08)
 				)
 			)
@@
 		)
 		(property "Value" "20k"
-			(at 0 1.43 0)
-			(layer "F.Fab")
-			(effects
-				(font
-					(size 1 1)
-					(thickness 0.15)
+			(at 2.1 0 0)
+			(unlocked yes)
+			(layer "F.Fab")
+			(effects
+				(font
+					(size 0.5 0.5)
+					(thickness 0.08)
 				)
 			)
@@
 		)
 		(property "Value" "48037-0001"
-			(at 3.26 18.965 90)
-			(layer "F.Fab")
-			(effects
-				(font
-					(size 1 1)
-					(thickness 0.15)
+			(at 0 0.4 90)
+			(unlocked yes)
+			(layer "F.Fab")
+			(effects
+				(font
+					(size 0.4 0.4)
+					(thickness 0.08)
 				)
 			)
@@
 		(attr through_hole)
 		(duplicate_pad_numbers_are_jumpers no)
-		(fp_line
-			(start -6 17.8)
-			(end 6 17.8)
-			(stroke
-				(width 0.127)
-				(type solid)
-			)
-			(layer "F.SilkS")
-		)
-		(fp_line
-			(start 6 17.8)
-			(end 6 2.75)
-			(stroke
-				(width 0.127)
-				(type solid)
-			)
-			(layer "F.SilkS")
-		)
-		(fp_line
-			(start -6 2.75)
-			(end -6 17.8)
-			(stroke
-				(width 0.127)
-				(type solid)
-			)
-			(layer "F.SilkS")
-		)
-		(fp_line
-			(start -6 2.75)
-			(end 6 2.75)
-			(stroke
-				(width 0.127)
-				(type solid)
-			)
-			(layer "F.SilkS")
-		)
-		(fp_line
-			(start 6 2.75)
-			(end 6 2)
-			(stroke
-				(width 0.127)
-				(type solid)
-			)
-			(layer "F.SilkS")
-		)
-		(fp_line
-			(start -6 2)
-			(end -6 2.75)
-			(stroke
-				(width 0.127)
-				(type solid)
-			)
-			(layer "F.SilkS")
-		)
 		(fp_circle
 			(center 3.5 -3.4)
@@
 					(size 0.32 0.32)
 					(thickness 0.15)
+				)
+			)
+		)
+		(fp_text user "${REFERENCE}"
+			(at 0 -1 90)
+			(unlocked yes)
+			(layer "F.Fab")
+			(effects
+				(font
+					(size 0.5 0.5)
+					(thickness 0.08)
 				)
 			)
@@
 		)
 		(property "Value" "110"
-			(at 0 1.43 270)
-			(layer "F.Fab")
-			(effects
-				(font
-					(size 1 1)
-					(thickness 0.15)
+			(at 2.05 0 0)
+			(unlocked yes)
+			(layer "F.Fab")
+			(effects
+				(font
+					(size 0.5 0.5)
+					(thickness 0.08)
 				)
 			)
@@
 		(tags "resistor")
 		(property "Reference" "R1"
-			(at 0.15 -1.15 90)
+			(at 0.35 -1.2 90)
 			(unlocked yes)
 			(layer "F.SilkS")
@@
 		)
 		(property "Value" "4.99k"
-			(at 0 1.43 270)
-			(layer "F.Fab")
-			(effects
-				(font
-					(size 1 1)
-					(thickness 0.15)
+			(at 0 -0.8 90)
+			(unlocked yes)
+			(layer "F.Fab")
+			(effects
+				(font
+					(size 0.5 0.5)
+					(thickness 0.08)
 				)
 			)
@@
 		(tags "capacitor")
 		(property "Reference" "C1"
-			(at -2 0 0)
+			(at -2 0.25 90)
 			(unlocked yes)
 			(layer "F.SilkS")
@@
 		)
 		(property "Value" "1u"
-			(at 0 1.43 180)
-			(layer "F.Fab")
-			(effects
-				(font
-					(size 1 1)
-					(thickness 0.15)
+			(at 2 0 90)
+			(unlocked yes)
+			(layer "F.Fab")
+			(effects
+				(font
+					(size 0.5 0.5)
+					(thickness 0.08)
 				)
 			)
@@
 		(tags "capacitor")
 		(property "Reference" "C5"
-			(at -1.2 -1.3 0)
+			(at -1.3 -2.12 90)
 			(unlocked yes)
 			(layer "F.SilkS")
@@
 		)
 		(property "Value" "1u"
-			(at 0 1.43 270)
-			(layer "F.Fab")
-			(effects
-				(font
-					(size 1 1)
-					(thickness 0.15)
+			(at 0 0.85 90)
+			(unlocked yes)
+			(layer "F.Fab")
+			(effects
+				(font
+					(size 0.5 0.5)
+					(thickness 0.08)
 				)
 			)
@@
 		)
 		(property "Value" "10u"
-			(at 0 1.43 270)
-			(layer "F.Fab")
-			(effects
-				(font
-					(size 1 1)
-					(thickness 0.15)
+			(at 0 0.85 90)
+			(unlocked yes)
+			(layer "F.Fab")
+			(effects
+				(font
+					(size 0.5 0.5)
+					(thickness 0.08)
 				)
 			)
@@
 		(layer "Edge.Cuts")
 	)
+	(gr_text "MP1 LED FLASHER"
+		(at 123.2 108.6 90)
+		(layer "B.SilkS")
+		(effects
+			(font
+				(size 0.8 0.8)
+				(thickness 0.12)
+			)
+			(justify mirror)
+		)
+	)
+	(gr_text "D. SHAH  ENGR 3430"
+		(at 124.4 108.6 90)
+		(layer "B.SilkS")
+		(effects
+			(font
+				(size 0.8 0.8)
+				(thickness 0.12)
+			)
+			(justify mirror)
+		)
+	)
+	(gr_text "REV A  2026-09"
+		(at 125.6 108.6 90)
+		(layer "B.SilkS")
+		(effects
+			(font
+				(size 0.8 0.8)
+				(thickness 0.12)
+			)
+			(justify mirror)
+		)
+	)
 	(segment
